Commit message: semi-working mulran parameters

File: config/robot.urdf.xacro (robot description, xacro)
@@ -33,3 +33,9 @@
     <origin xyz="0 0 0" rpy="0 0 0" />
   </joint>
+  <!-- <link name="world"/>
+    <joint name="world_joint" type="fixed">
+    <parent link="world"/>
+    <child link="base_link"/>
+    <origin xyz="0 0 0" rpy="0 0 0"/>
+  </joint> -->
 </robot>
